File: Hardware/CAN_Logger.sch (EAGLE design)
At the start: 56 parts, among them IC1 REG1117, Q1 8 MHz, U1 STM32F405XXSTM32F405XX, U4 MCP2551-E/SN, X2 22-23-2021, X4 22-23-2031, X5 MINI-USB-32005-301

Commit message: updated to hardware revision 2
Parts:
- removed C6: 0.1 u, rcl:C-EUC0603
- removed R1, R15: 22, resistor:R-US_R0603
- removed R16: 1 k, resistor:R-US_R0603
- removed R20: 4.7k, resistor:R-US_R0603
- removed U$2: MICROSD, adafruit:MICROSD
- removed X5: MINI-USB-32005-301, con-cypressindustries:MINI-USB-32005-301
- added U$1: NONAME_SD, uSD:NONAME_SD
- C1: value 0.1 u -> 100 nF
- C10, C22: value 20p -> 18 pF
- C15, C21: value 2u2 -> 2.2 uF
- C16, C17, C19, C20, C23, C7: value 100 n -> 100 nF
- C2, C5: value 10u -> 10 uF x 25V
- C4: value 1u -> 2.2 uF
- C8, C9: value 560 -> 560 pF
- IC1: value REG1117 -> NCP1117ST33T3G
- LED1: value (none) -> Red
- LED2: value (none) -> Blue
- LED3: value (none) -> Green
- Q1: value 8 MHz -> ABLS2-8.000MHZ
- R11, R12: value 20 -> 22
- R13, R4: value 4.7k -> 4.7 k
- R14: value 22 -> 0; device resistor:R-US_R0603 -> rcl:R-US_R0402
- U1: value STM32F405XXSTM32F405XX -> STM32F405RGT6
- U4: value MCP2551-E/SN -> SN65HVD232DR
Connections:
- removed net N$3: R1.1, U$2.CARD_DETECT
- removed net N$30: R16.2, U1.PA9
- removed net N$33: R15.2, X5.3
- removed net N$36: R14.2, X5.2
- removed net USB_VBUS: D2.A1, R16.1, R20.1, X5.1
- new net N$2: D2.A2, X2-2.S
- net +3V3: now also U$1.4; no longer U$2.VDD
- net GND: now also U$1.6, U$1.M1, U$1.M2, X2-1.S; no longer C6.2, R20.2, U$2.GND, U$2.GND1, U$2.VSS, X2-2.S, X5.5
- net MMC_NCD: no longer R1.2
- net N$10: now also R14.1; no longer R9.2
- net N$11: now also U$1.2; no longer U$2.CS
- net N$19: now also U$1.8; no longer U$2.DAT1
- net N$20: now also U$1.1; no longer U$2.DAT2
- net N$29: now also R14.2, R9.2; no longer D2.A2, X2-1.S
- net N$4: now also U$1.3; no longer U$2.DATA_IN
- net N$5: now also U$1.7; no longer U$2.DATA_OUT
- net N$6: now also U$1.5; no longer U$2.SCLK
- net N$9: no longer C6.1
- net USB_DM: no longer R14.1
- net USB_DP: no longer R15.1
Other:
- note removed: "Amphenol 101‑00660‑68‑6‑1‑ND"
- note removed: "replaced to SN65HVD232DR"
- moved on the sheet: C1, C2, R14, R2, R22, R23, R3, R5, R6, X2-1, X2-2

Commit message: additional configuartion options for start/stop logs implemented
start_on_power, circular_write, start_id, stop_id, start_on_CAN, stop_on_CAN, start_frame_to_name
Parts:
- R14: device rcl:R-US_R0402 -> rcl:R-US_R0201
Changed lines of the file:
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@@
 <grid distance="0.1" unitdist="inch" unit="inch" style="lines" multiple="1" display="no" altdistance="0.01" altunitdist="inch" altunit="inch"/>
 <layers>
-<layer number="1" name="Top" color="4" fill="1" visible="no" active="no"/>
-<layer number="2" name="Route2" color="1" fill="3" visible="no" active="no"/>
-<layer number="3" name="Route3" color="4" fill="3" visible="no" active="no"/>
-<layer number="4" name="Route4" color="1" fill="4" visible="no" active="no"/>
-<layer number="5" name="Route5" color="4" fill="4" visible="no" active="no"/>
-<layer number="6" name="Route6" color="1" fill="8" visible="no" active="no"/>
-<layer number="7" name="Route7" color="4" fill="8" visible="no" active="no"/>
-<layer number="8" name="Route8" color="1" fill="2" visible="no" active="no"/>
-<layer number="9" name="Route9" color="4" fill="2" visible="no" active="no"/>
-<layer number="10" name="Route10" color="1" fill="7" visible="no" active="no"/>
-<layer number="11" name="Route11" color="4" fill="7" visible="no" active="no"/>
-<layer number="12" name="Route12" color="1" fill="5" visible="no" active="no"/>
-<layer number="13" name="Route13" color="4" fill="5" visible="no" active="no"/>
-<layer number="14" name="Route14" color="1" fill="6" visible="no" active="no"/>
-<layer number="15" name="Route15" color="4" fill="6" visible="no" active="no"/>
-<layer number="16" name="Bottom" color="1" fill="1" visible="no" active="no"/>
-<layer number="17" name="Pads" color="2" fill="1" visible="no" active="no"/>
-<layer number="18" name="Vias" color="2" fill="1" visible="no" active="no"/>
-<layer number="19" name="Unrouted" color="6" fill="1" visible="no" active="no"/>
-<layer number="20" name="Dimension" color="15" fill="1" visible="no" active="no"/>
-<layer number="21" name="tPlace" color="7" fill="1" visible="no" active="no"/>
-<layer number="22" name="bPlace" color="7" fill="1" visible="no" active="no"/>
-<layer number="23" name="tOrigins" color="15" fill="1" visible="no" active="no"/>
-<layer number="24" name="bOrigins" color="15" fill="1" visible="no" active="no"/>
-<layer number="25" name="tNames" color="7" fill="1" visible="no" active="no"/>
-<layer number="26" name="bNames" color="7" fill="1" visible="no" active="no"/>
-<layer number="27" name="tValues" color="7" fill="1" visible="no" active="no"/>
-<layer number="28" name="bValues" color="7" fill="1" visible="no" active="no"/>
+<layer number="1" name="Top" color="4" fill="1" visible="yes" active="no"/>
+<layer number="2" name="Route2" color="1" fill="3" visible="yes" active="no"/>
+<layer number="3" name="Route3" color="4" fill="3" visible="yes" active="no"/>
+<layer number="4" name="Route4" color="1" fill="4" visible="yes" active="no"/>
+<layer number="5" name="Route5" color="4" fill="4" visible="yes" active="no"/>
+<layer number="6" name="Route6" color="1" fill="8" visible="yes" active="no"/>
+<layer number="7" name="Route7" color="4" fill="8" visible="yes" active="no"/>
+<layer number="8" name="Route8" color="1" fill="2" visible="yes" active="no"/>
+<layer number="9" name="Route9" color="4" fill="2" visible="yes" active="no"/>
+<layer number="10" name="Route10" color="1" fill="7" visible="yes" active="no"/>
+<layer number="11" name="Route11" color="4" fill="7" visible="yes" active="no"/>
+<layer number="12" name="Route12" color="1" fill="5" visible="yes" active="no"/>
+<layer number="13" name="Route13" color="4" fill="5" visible="yes" active="no"/>
+<layer number="14" name="Route14" color="1" fill="6" visible="yes" active="no"/>
+<layer number="15" name="Route15" color="4" fill="6" visible="yes" active="no"/>
+<layer number="16" name="Bottom" color="1" fill="1" visible="yes" active="no"/>
+<layer number="17" name="Pads" color="2" fill="1" visible="yes" active="no"/>
+<layer number="18" name="Vias" color="2" fill="1" visible="yes" active="no"/>
+<layer number="19" name="Unrouted" color="6" fill="1" visible="yes" active="no"/>
+<layer number="20" name="Dimension" color="15" fill="1" visible="yes" active="no"/>
+<layer number="21" name="tPlace" color="7" fill="1" visible="yes" active="no"/>
+<layer number="22" name="bPlace" color="7" fill="1" visible="yes" active="no"/>
+<layer number="23" name="tOrigins" color="15" fill="1" visible="yes" active="no"/>
+<layer number="24" name="bOrigins" color="15" fill="1" visible="yes" active="no"/>
+<layer number="25" name="tNames" color="7" fill="1" visible="yes" active="no"/>
+<layer number="26" name="bNames" color="7" fill="1" visible="yes" active="no"/>
+<layer number="27" name="tValues" color="7" fill="1" visible="yes" active="no"/>
+<layer number="28" name="bValues" color="7" fill="1" visible="yes" active="no"/>
 <layer number="29" name="tStop" color="7" fill="3" visible="no" active="no"/>
 <layer number="30" name="bStop" color="7" fill="6" visible="no" active="no"/>
@@
 <layer number="35" name="tGlue" color="7" fill="4" visible="no" active="no"/>
 <layer number="36" name="bGlue" color="7" fill="5" visible="no" active="no"/>
-<layer number="37" name="tTest" color="7" fill="1" visible="no" active="no"/>
-<layer number="38" name="bTest" color="7" fill="1" visible="no" active="no"/>
+<layer number="37" name="tTest" color="7" fill="1" visible="yes" active="no"/>
+<layer number="38" name="bTest" color="7" fill="1" visible="yes" active="no"/>
 <layer number="39" name="tKeepout" color="4" fill="11" visible="no" active="no"/>
 <layer number="40" name="bKeepout" color="1" fill="11" visible="no" active="no"/>
@@
 <layer number="44" name="Drills" color="7" fill="1" visible="no" active="no"/>
 <layer number="45" name="Holes" color="7" fill="1" visible="no" active="no"/>
-<layer number="46" name="Milling" color="3" fill="1" visible="no" active="no"/>
-<layer number="47" name="Measures" color="7" fill="1" visible="no" active="no"/>
-<layer number="48" name="Document" color="7" fill="1" visible="no" active="no"/>
-<layer number="49" name="Reference" color="7" fill="1" visible="no" active="no"/>
-<layer number="50" name="dxf" color="7" fill="1" visible="no" active="no"/>
-<layer number="51" name="tDocu" color="7" fill="1" visible="no" active="no"/>
-<layer number="52" name="bDocu" color="7" fill="1" visible="no" active="no"/>
-<layer number="53" name="tGND_GNDA" color="7" fill="9" visible="no" active="no"/>
-<layer number="54" name="bGND_GNDA" color="1" fill="9" visible="no" active="no"/>
-<layer number="56" name="wert" color="7" fill="1" visible="no" active="no"/>
-<layer number="57" name="tCAD" color="7" fill="1" visible="no" active="no"/>
-<layer number="59" name="tCarbon" color="7" fill="1" visible="no" active="no"/>
-<layer number="60" name="bCarbon" color="7" fill="1" visible="no" active="no"/>
+<layer number="46" name="Milling" color="3" fill="1" visible="yes" active="no"/>
+<layer number="47" name="Measures" color="7" fill="1" visible="yes" active="no"/>
+<layer number="48" name="Document" color="7" fill="1" visible="yes" active="no"/>
+<layer number="49" name="Reference" color="7" fill="1" visible="yes" active="no"/>
+<layer number="50" name="dxf" color="7" fill="1" visible="yes" active="no"/>
+<layer number="51" name="tDocu" color="7" fill="1" visible="yes" active="no"/>
+<layer number="52" name="bDocu" color="7" fill="1" visible="yes" active="no"/>
+<layer number="53" name="tGND_GNDA" color="7" fill="9" visible="yes" active="no"/>
+<layer number="54" name="bGND_GNDA" color="1" fill="9" visible="yes" active="no"/>
+<layer number="56" name="wert" color="7" fill="1" visible="yes" active="no"/>
+<layer number="57" name="tCAD" color="7" fill="1" visible="yes" active="no"/>
+<layer number="59" name="tCarbon" color="7" fill="1" visible="yes" active="no"/>
+<layer number="60" name="bCarbon" color="7" fill="1" visible="yes" active="no"/>
 <layer number="90" name="Modules" color="5" fill="1" visible="yes" active="yes"/>
 <layer number="91" name="Nets" color="2" fill="1" visible="yes" active="yes"/>
@@
 <part name="GND2" library="supply1" deviceset="GND" device=""/>
 <part name="+3V8" library="supply1" deviceset="+3V3" device=""/>
-<part name="R14" library="rcl" deviceset="R-US_" device="R0402" value="0"/>
+<part name="R14" library="rcl" deviceset="R-US_" device="R0201" value="0"/>
 <part name="U$1" library="uSD" deviceset="NONAME_SD" device=""/>
 <part name="GND3" library="supply1" deviceset="GND" device=""/>
